File: pcb/filter_bank.kicad_sch (KiCad schematic)
At the start: 18 parts, among them K1 G6K-2F-Y-DC5, K2 G6K-2F-Y-DC5, K3 G6K-2F-Y-DC5, K4 G6K-2F-Y-DC5, K5 G6K-2F-Y-DC5, K6 G6K-2F-Y-DC5, Q6 AO3400A, Q7 AO3400A, Q9 AO3400A

Commit message: Renumber all references monotonically 1..N per prefix; sync PCB silk labels and auto-named nets; ERC 0, DRC 0/0
Parts:
- renumbered D1 to D3, D2 to D5, D5 to D6, D3 to D7, D6 to D8, K4 to K2, K2 to K3, K5 to K4, K3 to K5, Q6 to Q5, Q7 to Q6, Q9 to Q7, R9 to R24, R10 to R25, R91 to R26
Changed lines of the file:
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@@
 		(on_board yes)
 		(dnp no)
-		(property "Reference" "D1"
+		(property "Reference" "D3"
 			(at 161.93 63.5 0)
 			(effects
@@
 			(project "OpenBeacon2"
 				(path "/046319a3-a6ce-4e59-a888-94e340127381/7b1c0f3e-4a51-4c1e-9f2a-0b5e1f1a2b01"
-					(reference "D1")
+					(reference "D3")
 					(unit 1)
 				)
@@
 		(on_board yes)
 		(dnp no)
-		(property "Reference" "#PWR917"
+		(property "Reference" "#PWR49"
 			(at 139.7 57.15 0)
 			(effects
@@
 			(project "OpenBeacon2"
 				(path "/046319a3-a6ce-4e59-a888-94e340127381/7b1c0f3e-4a51-4c1e-9f2a-0b5e1f1a2b01"
-					(reference "#PWR917")
+					(reference "#PWR49")
 					(unit 1)
 				)
@@
 		(on_board yes)
 		(dnp no)
-		(property "Reference" "K2"
+		(property "Reference" "K3"
 			(at 152.4 67.31 90)
 			(effects
@@
 			(project "OpenBeacon2"
 				(path "/046319a3-a6ce-4e59-a888-94e340127381/7b1c0f3e-4a51-4c1e-9f2a-0b5e1f1a2b01"
-					(reference "K2")
+					(reference "K3")
 					(unit 1)
 				)
@@
 		(on_board yes)
 		(dnp no)
-		(property "Reference" "D2"
+		(property "Reference" "D5"
 			(at 161.93 102.87 0)
 			(effects
@@
 			(project "OpenBeacon2"
 				(path "/046319a3-a6ce-4e59-a888-94e340127381/7b1c0f3e-4a51-4c1e-9f2a-0b5e1f1a2b01"
-					(reference "D2")
+					(reference "D5")
 					(unit 1)
 				)
@@
 		(on_board yes)
 		(dnp no)
-		(property "Reference" "#PWR918"
+		(property "Reference" "#PWR51"
 			(at 139.7 96.52 0)
 			(effects
@@
 			(project "OpenBeacon2"
 				(path "/046319a3-a6ce-4e59-a888-94e340127381/7b1c0f3e-4a51-4c1e-9f2a-0b5e1f1a2b01"
-					(reference "#PWR918")
+					(reference "#PWR51")
 					(unit 1)
 				)
@@
 		(on_board yes)
 		(dnp no)
-		(property "Reference" "K3"
+		(property "Reference" "K5"
 			(at 152.4 106.68 90)
 			(effects
@@
 			(project "OpenBeacon2"
 				(path "/046319a3-a6ce-4e59-a888-94e340127381/7b1c0f3e-4a51-4c1e-9f2a-0b5e1f1a2b01"
-					(reference "K3")
+					(reference "K5")
 					(unit 1)
 				)
@@
 		(on_board yes)
 		(dnp no)
-		(property "Reference" "D3"
+		(property "Reference" "D7"
 			(at 161.93 142.24 0)
 			(effects
@@
 			(project "OpenBeacon2"
 				(path "/046319a3-a6ce-4e59-a888-94e340127381/7b1c0f3e-4a51-4c1e-9f2a-0b5e1f1a2b01"
-					(reference "D3")
+					(reference "D7")
 					(unit 1)
 				)
@@
 		(on_board yes)
 		(dnp no)
-		(property "Reference" "#PWR919"
+		(property "Reference" "#PWR53"
 			(at 139.7 135.89 0)
 			(effects
@@
 			(project "OpenBeacon2"
 				(path "/046319a3-a6ce-4e59-a888-94e340127381/7b1c0f3e-4a51-4c1e-9f2a-0b5e1f1a2b01"
-					(reference "#PWR919")
+					(reference "#PWR53")
 					(unit 1)
 				)
@@
 		(on_board yes)
 		(dnp no)
-		(property "Reference" "K4"
+		(property "Reference" "K2"
 			(at 236.22 27.94 90)
 			(effects
@@
 			(project "OpenBeacon2"
 				(path "/046319a3-a6ce-4e59-a888-94e340127381/7b1c0f3e-4a51-4c1e-9f2a-0b5e1f1a2b01"
-					(reference "K4")
+					(reference "K2")
 					(unit 1)
 				)
@@
 		(on_board yes)
 		(dnp no)
-		(property "Reference" "#PWR920"
+		(property "Reference" "#PWR50"
 			(at 223.52 57.15 0)
 			(effects
@@
 			(project "OpenBeacon2"
 				(path "/046319a3-a6ce-4e59-a888-94e340127381/7b1c0f3e-4a51-4c1e-9f2a-0b5e1f1a2b01"
-					(reference "#PWR920")
+					(reference "#PWR50")
 					(unit 1)
 				)
@@
 		(on_board yes)
 		(dnp no)
-		(property "Reference" "K5"
+		(property "Reference" "K4"
 			(at 236.22 67.31 90)
 			(effects
@@
 			(project "OpenBeacon2"
 				(path "/046319a3-a6ce-4e59-a888-94e340127381/7b1c0f3e-4a51-4c1e-9f2a-0b5e1f1a2b01"
-					(reference "K5")
+					(reference "K4")
 					(unit 1)
 				)
@@
 		(on_board yes)
 		(dnp no)
-		(property "Reference" "D5"
+		(property "Reference" "D6"
 			(at 245.75 102.87 0)
 			(effects
@@
 			(project "OpenBeacon2"
 				(path "/046319a3-a6ce-4e59-a888-94e340127381/7b1c0f3e-4a51-4c1e-9f2a-0b5e1f1a2b01"
-					(reference "D5")
+					(reference "D6")
 					(unit 1)
 				)
@@
 		(on_board yes)
 		(dnp no)
-		(property "Reference" "#PWR921"
+		(property "Reference" "#PWR52"
 			(at 223.52 96.52 0)
 			(effects
@@
 			(project "OpenBeacon2"
 				(path "/046319a3-a6ce-4e59-a888-94e340127381/7b1c0f3e-4a51-4c1e-9f2a-0b5e1f1a2b01"
-					(reference "#PWR921")
+					(reference "#PWR52")
 					(unit 1)
 				)
@@
 		(on_board yes)
 		(dnp no)
-		(property "Reference" "D6"
+		(property "Reference" "D8"
 			(at 245.75 142.24 0)
 			(effects
@@
 			(project "OpenBeacon2"
 				(path "/046319a3-a6ce-4e59-a888-94e340127381/7b1c0f3e-4a51-4c1e-9f2a-0b5e1f1a2b01"
-					(reference "D6")
+					(reference "D8")
 					(unit 1)
 				)
@@
 		(on_board yes)
 		(dnp no)
-		(property "Reference" "#PWR922"
+		(property "Reference" "#PWR54"
 			(at 223.52 135.89 0)
 			(effects
@@
 			(project "OpenBeacon2"
 				(path "/046319a3-a6ce-4e59-a888-94e340127381/7b1c0f3e-4a51-4c1e-9f2a-0b5e1f1a2b01"
-					(reference "#PWR922")
+					(reference "#PWR54")
 					(unit 1)
 				)
@@
 		(on_board yes)
 		(dnp no)
-		(property "Reference" "Q6"
+		(property "Reference" "Q5"
 			(at 45.72 168.91 0)
 			(effects
@@
 			(project "OpenBeacon2"
 				(path "/046319a3-a6ce-4e59-a888-94e340127381/7b1c0f3e-4a51-4c1e-9f2a-0b5e1f1a2b01"
-					(reference "Q6")
+					(reference "Q5")
 					(unit 1)
 				)
@@
 		(on_board yes)
 		(dnp no)
-		(property "Reference" "R9"
+		(property "Reference" "R24"
 			(at 28.575 171.45 0)
 			(effects
@@
 			(project "OpenBeacon2"
 				(path "/046319a3-a6ce-4e59-a888-94e340127381/7b1c0f3e-4a51-4c1e-9f2a-0b5e1f1a2b01"
-					(reference "R9")
+					(reference "R24")
 					(unit 1)
 				)
@@
 		(on_board yes)
 		(dnp no)
-		(property "Reference" "#PWR923"
+		(property "Reference" "#PWR55"
 			(at 30.48 175.26 0)
 			(effects
@@
 			(project "OpenBeacon2"
 				(path "/046319a3-a6ce-4e59-a888-94e340127381/7b1c0f3e-4a51-4c1e-9f2a-0b5e1f1a2b01"
-					(reference "#PWR923")
+					(reference "#PWR55")
 					(unit 1)
 				)
@@
 		(on_board yes)
 		(dnp no)
-		(property "Reference" "#PWR924"
+		(property "Reference" "#PWR56"
 			(at 43.18 175.26 0)
 			(effects
@@
 			(project "OpenBeacon2"
 				(path "/046319a3-a6ce-4e59-a888-94e340127381/7b1c0f3e-4a51-4c1e-9f2a-0b5e1f1a2b01"
-					(reference "#PWR924")
+					(reference "#PWR56")
 					(unit 1)
 				)
@@
 		(on_board yes)
 		(dnp no)
-		(property "Reference" "Q7"
+		(property "Reference" "Q6"
 			(at 93.98 168.91 0)
 			(effects
@@
 			(project "OpenBeacon2"
 				(path "/046319a3-a6ce-4e59-a888-94e340127381/7b1c0f3e-4a51-4c1e-9f2a-0b5e1f1a2b01"
-					(reference "Q7")
+					(reference "Q6")
 					(unit 1)
 				)
@@
 		(on_board yes)
 		(dnp no)
-		(property "Reference" "R10"
+		(property "Reference" "R25"
 			(at 76.835 171.45 0)
 			(effects
@@
 			(project "OpenBeacon2"
 				(path "/046319a3-a6ce-4e59-a888-94e340127381/7b1c0f3e-4a51-4c1e-9f2a-0b5e1f1a2b01"
-					(reference "R10")
+					(reference "R25")
 					(unit 1)
 				)
@@
 		(on_board yes)
 		(dnp no)
-		(property "Reference" "#PWR925"
+		(property "Reference" "#PWR57"
 			(at 78.74 175.26 0)
 			(effects
@@
 			(project "OpenBeacon2"
 				(path "/046319a3-a6ce-4e59-a888-94e340127381/7b1c0f3e-4a51-4c1e-9f2a-0b5e1f1a2b01"
-					(reference "#PWR925")
+					(reference "#PWR57")
 					(unit 1)
 				)
@@
 		(on_board yes)
 		(dnp no)
-		(property "Reference" "#PWR926"
+		(property "Reference" "#PWR58"
 			(at 91.44 175.26 0)
 			(effects
@@
 			(project "OpenBeacon2"
 				(path "/046319a3-a6ce-4e59-a888-94e340127381/7b1c0f3e-4a51-4c1e-9f2a-0b5e1f1a2b01"
-					(reference "#PWR926")
+					(reference "#PWR58")
 					(unit 1)
 				)
@@
 		(in_pos_files yes)
 		(dnp no)
-		(property "Reference" "Q9"
+		(property "Reference" "Q7"
 			(at 93.98 184.15 0)
 			(effects (font (size 1.27 1.27)) (justify left))
@@
 			(project "OpenBeacon2"
 				(path "/046319a3-a6ce-4e59-a888-94e340127381/7b1c0f3e-4a51-4c1e-9f2a-0b5e1f1a2b01"
-					(reference "Q9")
+					(reference "Q7")
 					(unit 1)
 				)
@@
 		(in_pos_files yes)
 		(dnp no)
-		(property "Reference" "R91"
+		(property "Reference" "R26"
 			(at 73.2 187.4 0)
 			(effects (font (size 1.27 1.27)) (justify left))
@@
 			(project "OpenBeacon2"
 				(path "/046319a3-a6ce-4e59-a888-94e340127381/7b1c0f3e-4a51-4c1e-9f2a-0b5e1f1a2b01"
-					(reference "R91")
+					(reference "R26")
 					(unit 1)
 				)
@@
 		(in_pos_files yes)
 		(dnp no)
-		(property "Reference" "#PWR1991"
+		(property "Reference" "#PWR59"
 			(at 81.28 189.23 0)
 			(hide yes)
@@
 			(project "OpenBeacon2"
 				(path "/046319a3-a6ce-4e59-a888-94e340127381/7b1c0f3e-4a51-4c1e-9f2a-0b5e1f1a2b01"
-					(reference "#PWR1991")
+					(reference "#PWR59")
 					(unit 1)
 				)
@@
 		(in_pos_files yes)
 		(dnp no)
-		(property "Reference" "#PWR1992"
+		(property "Reference" "#PWR60"
 			(at 93.98 189.23 0)
 			(hide yes)
@@
 			(project "OpenBeacon2"
 				(path "/046319a3-a6ce-4e59-a888-94e340127381/7b1c0f3e-4a51-4c1e-9f2a-0b5e1f1a2b01"
-					(reference "#PWR1992")
+					(reference "#PWR60")
 					(unit 1)
 				)
